File: U23_2012.brd (EAGLE design)
At the start: 150 x 100 mm, 68 parts, among them T1 BC337, X2 J1006F01P

Commit message: fixes wrong named ground plane
committed to seed studio, rev_1.1_u23_final
adds committed zip file
Routing:
- added copper zone on layer 16, net GND
- removed copper zone on layer 16, net N$21
Other:
- board text added: "No: 61351"
